Commit message: Write actually sane config files

File: urdf/rover.urdf.xacro (robot description, xacro)
@@ -1,4 +1,12 @@
 <?xml version="1.0"?>
 <robot xmlns:xacro="http://www.ros.org/wiki/xacro" name="rover">
-  <!-- TODO: design robot-->
+  <transmission name="rover_transmission" />
+    <type>transmission_interface/SimpleTransmission</type>
+    <joint name="rover_joint_front_left">
+      <hardwareInterface>VelocityJointInterface</hardwareInterface>
+    </joint>
+    <actuator name="rover_wheel_front_left">
+      <mechanicalReduction>1</mechanicalReduction>
+    </actuator>
+  </transmission>
 </robot>

Commit message: Finish the URDF file

File: urdf/rover.urdf.xacro (robot description, xacro)
@@ -1,5 +1,5 @@
 <?xml version="1.0"?>
 <robot xmlns:xacro="http://www.ros.org/wiki/xacro" name="rover">
-  <transmission name="rover_transmission" />
+  <transmission name="rover_transmission_front_left" />
     <type>transmission_interface/SimpleTransmission</type>
     <joint name="rover_joint_front_left">
@@ -10,3 +10,30 @@
     </actuator>
   </transmission>
+  <transmission name="rover_transmission_front_right" />
+    <type>transmission_interface/SimpleTransmission</type>
+    <joint name="rover_joint_front_right">
+      <hardwareInterface>VelocityJointInterface</hardwareInterface>
+    </joint>
+    <actuator name="rover_wheel_front_right">
+      <mechanicalReduction>1</mechanicalReduction>
+    </actuator>
+  </transmission>
+  <transmission name="rover_transmission_back_right" />
+    <type>transmission_interface/SimpleTransmission</type>
+    <joint name="rover_joint_back_left">
+      <hardwareInterface>VelocityJointInterface</hardwareInterface>
+    </joint>
+    <actuator name="rover_wheel_back_left">
+      <mechanicalReduction>1</mechanicalReduction>
+    </actuator>
+  </transmission>
+  <transmission name="rover_transmission_back_right" />
+    <type>transmission_interface/SimpleTransmission</type>
+    <joint name="rover_joint_back_right">
+      <hardwareInterface>VelocityJointInterface</hardwareInterface>
+    </joint>
+    <actuator name="rover_wheel_back_right">
+      <mechanicalReduction>1</mechanicalReduction>
+    </actuator>
+  </transmission>
 </robot>

Commit message: Additional xacro changes

File: urdf/rover.urdf.xacro (robot description, xacro)
@@ -1,4 +1,25 @@
 <?xml version="1.0"?>
 <robot xmlns:xacro="http://www.ros.org/wiki/xacro" name="rover">
+  <link name="rover_link_front_left" />
+  <link name="rover_link_front_right" />
+  <link name="rover_link_back_left" />
+  <link name="rover_link_back_right" />
+  <link name="rover_link_base" />
+  <joint name="rover_joint_front_left" type="continuous">
+    <parent link="rover_link_base" />
+    <child link="rover_link_front_left" />
+  </joint>
+  <joint name="rover_joint_front_right" type="continuous">
+    <parent link="rover_link_base" />
+    <child link="rover_link_front_right" />
+  </joint>
+  <joint name="rover_joint_back_left" type="continuous">
+    <parent link="rover_link_base" />
+    <child link="rover_link_back_left" />
+  </joint>
+  <joint name="rover_joint_back_right" type="continuous">
+    <parent link="rover_link_base" />
+    <child link="rover_link_back_right" />
+  </joint>
   <transmission name="rover_transmission_front_left">
     <type>transmission_interface/SimpleTransmission</type>
